File: hardware/openstint-transponder.kicad_pcb (KiCad board)
At the start: 4 copper layers, 18 x 15 mm, 37 parts, among them J1 V+, J2 V-, Q1 PMGD280UN, U1 ATtiny1616-M, U2 10 MHz, U3 SPX3819M5-L-3-3

Commit message: v2 transponder - initial commit
Other:
- board size 18 x 15 mm -> 18.5 x 15 mm
Changed lines of the file:
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@@
 			)
 		)
+		(property "JLCPCB_CORRECTION" "0; 0; 180"
+			(at 0 0 180)
+			(unlocked yes)
+			(layer "F.Fab")
+			(hide yes)
+			(effects
+				(font
+					(size 1 1)
+					(thickness 0.15)
+				)
+			)
+		)
 		(sheetname "/")
 		(sheetfile "openstint-transponder.kicad_sch")
@@
 			)
 		)
+		(property "JLCPCB_CORRECTION" "0; 0; 180"
+			(at 0 0 180)
+			(unlocked yes)
+			(layer "F.Fab")
+			(hide yes)
+			(effects
+				(font
+					(size 1 1)
+					(thickness 0.15)
+				)
+			)
+		)
 		(property ki_fp_filters "LED* LED_SMD:* LED_THT:*")
 		(sheetname "/")
@@
 			)
 		)
+		(property "JLCPCB_CORRECTION" "0; 0; 270"
+			(at 0 0 270)
+			(unlocked yes)
+			(layer "F.Fab")
+			(hide yes)
+			(effects
+				(font
+					(size 1 1)
+					(thickness 0.15)
+				)
+			)
+		)
 		(property ki_fp_filters "VQFN*1EP*3x3mm*P0.4mm*")
 		(sheetname "/")
@@
 			)
 		)
-		(property "Datasheet" "https://jlcpcb.com/api/file/downloadByFileSystemAccessId/8590197686655098880"
+		(property "Datasheet" "https://jlcpcb.com/api/file/downloadByFileSystemAccessId/8613786702142062592"
 			(at 0 0 90)
 			(layer "F.Fab")
@@
 			)
 		)
-		(property "LCSC" "C2901558"
+		(property "LCSC" "C2831380"
 			(at 0 0 90)
 			(unlocked yes)
@@
 			)
 		)
+		(property "JLCPCB_CORRECTION" "0; 0; 270"
+			(at 0 0 180)
+			(unlocked yes)
+			(layer "F.Fab")
+			(hide yes)
+			(effects
+				(font
+					(size 1 1)
+					(thickness 0.15)
+				)
+			)
+		)
 		(property ki_fp_filters "SOT?23*")
 		(sheetname "/")
@@
 		(net 32)
 	)
+	(gr_circle
+		(center 146.7 108)
+		(end 146.65 108.1)
+		(stroke
+			(width 0.1)
+			(type solid)
+		)
+		(fill yes)
+		(layer "F.SilkS")
+	)
 	(gr_arc
 		(start 131.2 109.1)
@@
 	)
 	(gr_line
-		(start 130 95.5)
-		(end 130 109.5)
+		(start 129.75 95.5)
+		(end 129.75 109.5)
 		(stroke
 			(width 0.05)
@@
 	)
 	(gr_arc
-		(start 148 109.5)
-		(mid 147.853553 109.853553)
-		(end 147.5 110)
+		(start 130.25 110)
+		(mid 129.896447 109.853553)
+		(end 129.75 109.5)
 		(stroke
 			(width 0.05)
@@
 		(layer "Edge.Cuts")
 	)
-	(gr_arc
-		(start 130.5 110)
-		(mid 130.146447 109.853553)
-		(end 130 109.5)
+	(gr_line
+		(start 148.25 109.5)
+		(end 148.25 95.5)
 		(stroke
 			(width 0.05)
@@
 	)
 	(gr_line
-		(start 148 109.5)
-		(end 148 95.5)
+		(start 130.25 110)
+		(end 147.75 110)
 		(stroke
 			(width 0.05)
@@
 		(layer "Edge.Cuts")
 	)
-	(gr_line
-		(start 130.5 110)
-		(end 147.5 110)
+	(gr_arc
+		(start 147.75 95)
+		(mid 148.103553 95.146447)
+		(end 148.25 95.5)
 		(stroke
 			(width 0.05)
@@
 	)
 	(gr_arc
-		(start 147.5 95)
-		(mid 147.853553 95.146447)
-		(end 148 95.5)
+		(start 129.75 95.5)
+		(mid 129.896447 95.146447)
+		(end 130.25 95)
 		(stroke
 			(width 0.05)
@@
 	)
 	(gr_arc
-		(start 130 95.5)
-		(mid 130.146447 95.146447)
-		(end 130.5 95)
+		(start 148.25 109.5)
+		(mid 148.103553 109.853553)
+		(end 147.75 110)
 		(stroke
 			(width 0.05)
@@
 	)
 	(gr_line
-		(start 130.5 95)
-		(end 147.5 95)
+		(start 130.25 95)
+		(end 147.75 95)
 		(stroke
 			(width 0.05)

Commit message: spin v2
Parts:
- removed C10, C2: 100n, Capacitor_SMD:C_0402_1005Metric
- removed C11: 1n, Capacitor_SMD:C_0402_1005Metric
- removed TP2: TestPoint, TestPoint:TestPoint_Pad_D1.0mm
- added R10: 22, Resistor_SMD:R_0402_1005Metric, F.Cu at (133.2, 105.1)
- added R11: 22, Resistor_SMD:R_0402_1005Metric, F.Cu at (133.3, 99.9)
- added R8: 10, Resistor_SMD:R_0402_1005Metric, F.Cu at (133.2, 103.0)
- added R9: 10, Resistor_SMD:R_0402_1005Metric, F.Cu at (133.2, 102.0)
- added TP5: VTG, TestPoint:TestPoint_Pad_D1.0mm, B.Cu at (145.9, 99.6)
- C13, C14: value 22p -> 33p
- C5: value 10n -> 100n
- C6: value 1n -> 1800p/C0G
- R3, R4: value 22 -> 0
- TP1: value TestPoint -> UDPI
- TP3: value TestPoint -> VDDA
- TP4: value TestPoint -> GND
- U1: value ATtiny1616-M -> ATtiny816/1616
- moved D1 8.59 mm to (132.1, 108.6)
- moved R5 8.00 mm to (134.8, 108.6), turned to 180 degrees
- moved R6 5.29 mm to (136.2, 100.2), turned to 0 degrees
- moved R7 3.91 mm to (136.0, 104.8), turned to 180 degrees
- moved TP1 2.54 mm to (145.9, 104.7)
- moved TP4 2.54 mm to (145.9, 102.1)
- moved R4 2.27 mm to (132.7, 98.8), turned to 0 degrees
- moved R3 2.16 mm to (132.7, 106.2), turned to 0 degrees
- moved R2 1.78 mm to (136.0, 105.9)
- moved R1 1.58 mm to (136.0, 107.0), turned to 180 degrees
- moved Q1 1.46 mm to (135.7, 102.6), turned to -90 degrees
- moved C15 1.23 mm to (132.7, 107.2)
- moved C1 1.18 mm to (132.7, 97.7)
- moved C6 1.02 mm to (130.7, 102.5)
- moved C14 1.01 mm to (133.3, 100.9)
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Connections:
- C13 pad 1: GND -> Net-(C13-Pad1)
- C14 pad 2: GND -> Net-(C14-Pad2)
- Q1 pad 3: /A- -> /D-
- Q1 pad 6: /A+ -> /D+
- U1 pad 10: unconnected-(U1-PB4-Pad10) -> /~{BLINKY}
- U1 pad 20: /UART0TXD -> unconnected-(U1-PA1-Pad20)
- U1 pad 5: /ANT+ -> /ANT-
- U1 pad 6: /~{BLINKY} -> unconnected-(U1-PA5-Pad6)
- U1 pad 8: /ANT- -> /ANT+
Routing:
- net GND: track 78.9 -> 69.8 mm, vias 6 -> 11
- net /~{BLINKY}: track 10.0 -> 2.50 mm, vias 2 -> 0
- net /UART0TXD: track 7.00 -> 0.00 mm, vias 2 -> 0
- net /GANT+: track 4.29 -> 11.0 mm, vias 0 -> 2
- net +3.3V: track 43.8 -> 50.1 mm
- net /GANT-: track 9.20 -> 3.10 mm, vias 2 -> 0
- net /A-: track 9.25 -> 5.59 mm, vias 3 -> 2
- net /D+: track 0.00 -> 3.14 mm
- net /D-: track 0.00 -> 1.51 mm
- net /UDPI: track 7.81 -> 6.43 mm, vias 2 -> 1
- net Net-(C14-Pad2): track 0.00 -> 1.06 mm
- net Net-(C13-Pad1): track 0.00 -> 1.06 mm
- net /ANT-: track 1.29 -> 2.06 mm
- net /A+: track 5.69 -> 5.11 mm
Other:
- board text added: "VTG"
- board text removed: "TxD"
