File: hardware/openstint-transponder.kicad_pcb (KiCad board)
At the start: 4 copper layers, 18.5 x 15 mm, 39 parts, among them J1 V+, J2 V-, Q1 PMGD280UN, U1 ATtiny816/1616, U2 10 MHz, U3 SPX3819M5-L-3-3

Commit message: Fix UPDI label spelling
Signed-off-by: Voyagerroc-Pro <330935573+Voyagerroc-Pro@users.noreply.github.com>
Parts:
- TP1: value UDPI -> UPDI
Connections:
- net /UDPI renamed /UPDI
Other:
- board text added: "UPDI"
- board text removed: "UDPI"
Changed lines of the file:
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@@
 	(net 13 "/ANT+")
 	(net 14 "/ANT-")
-	(net 15 "/UDPI")
+	(net 15 "/UPDI")
 	(net 16 "unconnected-(U1-PB3-Pad11)")
 	(net 17 "unconnected-(U1-PA2-Pad1)")
@@
 			(layers "F.Cu" "F.Mask" "F.Paste")
 			(roundrect_rratio 0.25)
-			(net 15 "/UDPI")
+			(net 15 "/UPDI")
 			(pinfunction "~{RESET}/PA0")
 			(pintype "bidirectional")
@@
 			)
 		)
-		(property "Value" "UDPI"
+		(property "Value" "UPDI"
 			(at 0 -1.55 90)
 			(layer "B.Fab")
@@
 			(size 1 1)
 			(layers "B.Cu" "B.Mask")
-			(net 15 "/UDPI")
+			(net 15 "/UPDI")
 			(pinfunction "1")
 			(pintype "passive")
@@
 		)
 	)
-	(gr_text "UDPI"
+	(gr_text "UPDI"
 		(at 145.35 105.4 0)
 		(layer "B.SilkS")
