File: hardware/openstint-transponder.kicad_sch (KiCad schematic)
At the start: 40 parts, among them J1 V+, J2 V-, Q1 PMGD280UN, U1 ATtiny816/1616, U2 10 MHz, U3 SPX3819M5-L-3-3

Commit message: Fix UPDI label spelling
Signed-off-by: Voyagerroc-Pro <330935573+Voyagerroc-Pro@users.noreply.github.com>
Parts:
- TP1: value UDPI -> UPDI
Connections:
- net UDPI renamed UPDI
Changed lines of the file:
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@@
 		)
 	)
-	(label "UDPI"
+	(label "UPDI"
 		(at 119.38 40.64 180)
 		(effects
@@
 		)
 	)
-	(label "UDPI"
+	(label "UPDI"
 		(at 35.56 110.49 180)
 		(effects
@@
 			)
 		)
-		(property "Value" "UDPI"
+		(property "Value" "UPDI"
 			(at 24.638 107.95 90)
 			(effects
